Commit message: Task 2.1: Spawned with Color in Gazebo

File: urdf/sp_1.urdf.xacro (robot description, xacro)
@@ -3,6 +3,46 @@
      Commit Version: 1.6.0-4-g7f85cfe  Build Version: 1.6.7995.38578
      For more information, please see http://wiki.ros.org/sw_urdf_exporter -->
-<robot
-  name="sp_1">
+<robot xmlns:xacro="http://wiki.ros.org/xacro"  name="sp_1">
+<xacro:macro name="link_color">
+  <visual>
+    <material>
+      <ambient>0.501960784313725 1 0.501960784313725 1</ambient>
+      <diffuse>0.501960784313725 1 0.501960784313725 1</diffuse>
+      <specular>0.1 0.1 0.1 1</specular>
+      <emissive>0 0 0 0</emissive>
+    </material>
+  </visual>
+</xacro:macro>
+<xacro:macro name="base_color">
+  <visual>
+    <material>
+      <ambient>0 0 0 1</ambient>
+      <diffuse>0 0 0 1</diffuse>
+      <specular>0.1 0.1 0.1 1</specular>
+      <emissive>0 0 0 0</emissive>
+    </material>
+  </visual>
+</xacro:macro>
+<xacro:macro name="link2_color">
+  <visual>
+    <material>
+      <ambient>0.250980392156863 0.250980392156863 0.250980392156863 1</ambient>
+      <diffuse>0.250980392156863 0.250980392156863 0.250980392156863 1</diffuse>
+      <specular>0.1 0.1 0.1 1</specular>
+      <emissive>0 0 0 0</emissive>
+    </material>
+  </visual>
+</xacro:macro>
+<link
+    name="dummy_link">
+    <pose>0 0 0 0 0 0</pose>
+  </link>
+  <joint
+    name="dummy_joint" type="fixed">
+    <parent
+      link="dummy_link" />
+    <child
+      link="base_link" />
+  </joint>
   <link
     name="base_link">
@@ -509,3 +549,33 @@
       velocity="0" />
   </joint>
+  <gazebo reference="link_3">
+    <xacro:link_color />
+  </gazebo>
+  <gazebo reference="link_5">
+    <xacro:link_color />
+  </gazebo>
+  <gazebo reference="link_7">
+    <xacro:link_color />
+  </gazebo>
+  <!-- <gazebo reference="end_effector">
+    <xacro:link_color />
+  </gazebo> -->
+  <gazebo reference="base_link">
+    <xacro:base_color />
+  </gazebo>
+  <gazebo reference="link_1">
+    <xacro:link2_color />
+  </gazebo>
+  <gazebo reference="link_2">
+    <xacro:link2_color />
+  </gazebo>
+  <gazebo reference="link_4">
+    <xacro:link2_color />
+  </gazebo>
+  <gazebo reference="link_6">
+    <xacro:link2_color />
+  </gazebo>
+  <gazebo reference="end_effector">
+    <xacro:link2_color />
+  </gazebo>
 </robot>

Commit message: Task 2.2: Added Controllers

File: urdf/sp_1.urdf.xacro (robot description, xacro)
@@ -549,4 +549,92 @@
       velocity="0" />
   </joint>
+<!-- Transmission -->
+  <transmission name="trans_link1">
+    <type>transmission_interface/SimpleTransmission</type>
+    <joint name="joint_1">
+      <hardwareInterface>hardware_interface/EffortJointInterface</hardwareInterface>
+    </joint>
+    <actuator name="motor_link1">
+      <hardwareInterface>hardware_interface/EffortJointInterface</hardwareInterface>
+      <mechanicalReduction>1</mechanicalReduction>
+    </actuator>
+  </transmission>
+  <transmission name="trans_link2">
+    <type>transmission_interface/SimpleTransmission</type>
+    <joint name="joint_2">
+      <hardwareInterface>hardware_interface/EffortJointInterface</hardwareInterface>
+    </joint>
+    <actuator name="motor_link2">
+      <hardwareInterface>hardware_interface/EffortJointInterface</hardwareInterface>
+      <mechanicalReduction>1</mechanicalReduction>
+    </actuator>
+  </transmission>
+  <transmission name="trans_link3">
+    <type>transmission_interface/SimpleTransmission</type>
+    <joint name="joint_3">
+      <hardwareInterface>hardware_interface/EffortJointInterface</hardwareInterface>
+    </joint>
+    <actuator name="motor_link3">
+      <hardwareInterface>hardware_interface/EffortJointInterface</hardwareInterface>
+      <mechanicalReduction>1</mechanicalReduction>
+    </actuator>
+  </transmission>
+  <transmission name="trans_link4">
+    <type>transmission_interface/SimpleTransmission</type>
+    <joint name="joint_4">
+      <hardwareInterface>hardware_interface/EffortJointInterface</hardwareInterface>
+    </joint>
+    <actuator name="motor_link4">
+      <hardwareInterface>hardware_interface/EffortJointInterface</hardwareInterface>
+      <mechanicalReduction>1</mechanicalReduction>
+    </actuator>
+  </transmission>
+  <transmission name="trans_link5">
+    <type>transmission_interface/SimpleTransmission</type>
+    <joint name="joint_5">
+      <hardwareInterface>hardware_interface/EffortJointInterface</hardwareInterface>
+    </joint>
+    <actuator name="motor_link5">
+      <hardwareInterface>hardware_interface/EffortJointInterface</hardwareInterface>
+      <mechanicalReduction>1</mechanicalReduction>
+    </actuator>
+  </transmission>
+  <transmission name="trans_link6">
+    <type>transmission_interface/SimpleTransmission</type>
+    <joint name="joint_6">
+      <hardwareInterface>hardware_interface/EffortJointInterface</hardwareInterface>
+    </joint>
+    <actuator name="motor_link6">
+      <hardwareInterface>hardware_interface/EffortJointInterface</hardwareInterface>
+      <mechanicalReduction>1</mechanicalReduction>
+    </actuator>
+  </transmission>
+  <transmission name="trans_link7">
+    <type>transmission_interface/SimpleTransmission</type>
+    <joint name="joint_7">
+      <hardwareInterface>hardware_interface/EffortJointInterface</hardwareInterface>
+    </joint>
+    <actuator name="motor_link7">
+      <hardwareInterface>hardware_interface/EffortJointInterface</hardwareInterface>
+      <mechanicalReduction>1</mechanicalReduction>
+    </actuator>
+  </transmission>
+  <transmission name="trans_link8">
+    <type>transmission_interface/SimpleTransmission</type>
+    <joint name="joint_8">
+      <hardwareInterface>hardware_interface/EffortJointInterface</hardwareInterface>
+    </joint>
+    <actuator name="motor_link8">
+      <hardwareInterface>hardware_interface/EffortJointInterface</hardwareInterface>
+      <mechanicalReduction>1</mechanicalReduction>
+    </actuator>
+  </transmission>
+  <gazebo>
+    <plugin filename="libgazebo_ros_control.so" name="gazebo_ros_control">
+      <robotNamespace>/sp_1</robotNamespace>
+      <robotSimType>gazebo_ros_control/DefaultRobotHWSim</robotSimType>
+      <legacyModeNS>true</legacyModeNS>
+    </plugin>
+  </gazebo>
   <gazebo reference="link_3">
     <xacro:link_color />
@@ -558,7 +646,4 @@
     <xacro:link_color />
   </gazebo>
-  <!-- <gazebo reference="end_effector">
-    <xacro:link_color />
-  </gazebo> -->
   <gazebo reference="base_link">
     <xacro:base_color />
